Commit message: worked on the onshape export

File: onshape_to_robot/old_finger_edited/robot.urdf (robot description, URDF)
Before this commit: robot onshape, 3 links, 2 joints
Links:
- link part_1: mass 0 -> 0.0694721
- link part_2: mass 0 -> 0.086143
- link part_3: mass 0 -> 0.0603626
Joints:
- removed joint base
- removed joint notbase
- added joint rev1: type revolute, parent part_1, child part_2, origin xyz=-0.00893093 -0.0168919 0.0093023 rpy=-1.5708 4.39586e-16 -2.39529e-25, axis 0 0 1, limit lower=0 upper=1.5708 effort=1 velocity=20
- added joint rev2: type revolute, parent part_2, child part_3, origin xyz=-8.67362e-18 0.0445 -0.00675 rpy=3.14159 -2.39529e-25 -4.39586e-16, axis 0 0 1, limit lower=-1.5708 upper=0 effort=1 velocity=20
